File: EAGLE/gteo/Esquema.brd (EAGLE design)
At the start: 100 x 80 mm, 6 parts

Commit message: feat: add 3d model
Parts:
- added DIODO1: 1N4004, diode:DO41-10
Connections:
- new net 5V: WEMOS.JP2.8
- net N$5: now also DIODO1.A; no longer CONTROLBATERIA.B+
- net N$7: now also CONTROLBATERIA.B+, DIODO1.C; no longer CONTROLBATERIA.OUT+, WEMOS.JP2.8
- net N$8: now also CONTROLBATERIA.OUT+
Changed lines of the file:
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@@
 <attribute name="VALUE" x="87.63" y="59.69" size="1.27" layer="27" align="top-center"/>
+</element>
+<element name="DIODO1" library="diode" library_urn="urn:adsk.eagle:library:210" package="DO41-10" package3d_urn="urn:adsk.eagle:package:43336/1" value="1N4004" x="85.09" y="26.67" smashed="yes">
+<attribute name="NAME" x="83.058" y="28.321" size="1.27" layer="25" ratio="10"/>
+<attribute name="VALUE" x="83.058" y="23.876" size="1.27" layer="27" ratio="10"/>
 </element>
 </elements>
@@
 <wire x1="27.305" y1="27.305" x2="71.12" y2="55.245" width="0" layer="19" extent="1-1"/>
 </signal>
-<signal name="N$5">
-<contactref element="CONTROLBATERIA" pad="B+"/>
-<contactref element="BATERIA" pad="PWR@1"/>
-<wire x1="38.1" y1="27.305" x2="77.618" y2="10.17" width="0" layer="19" extent="1-1"/>
-</signal>
 <signal name="N$6">
 <contactref element="CONTROLBATERIA" pad="B-"/>
@@
 <wire x1="16.362" y1="10.15" x2="30.48" y2="27.305" width="0" layer="19" extent="1-1"/>
 </signal>
-<signal name="N$7">
-<contactref element="CONTROLBATERIA" pad="OUT+"/>
-<contactref element="WEMOS" pad="JP2.8"/>
-<wire x1="41.275" y1="27.305" x2="71.12" y2="52.705" width="0" layer="19" extent="1-1"/>
-</signal>
 <signal name="N$8">
 <contactref element="WEMOS" pad="JP1.8"/>
 <contactref element="SENSOR" pad="1"/>
+<contactref element="CONTROLBATERIA" pad="OUT+"/>
 <wire x1="48.26" y1="52.705" x2="82.55" y2="69.85" width="0" layer="19" extent="1-1"/>
+<wire x1="41.275" y1="27.305" x2="48.26" y2="52.705" width="0" layer="19" extent="1-1"/>
 </signal>
 <signal name="N$9">
@@
 <wire x1="40.64" y1="55.88" x2="41.275" y2="50.165" width="0" layer="19" extent="1-1"/>
 </signal>
+<signal name="5V">
+<contactref element="WEMOS" pad="JP2.8"/>
+</signal>
+<signal name="N$5">
+<contactref element="BATERIA" pad="PWR@1"/>
+<contactref element="DIODO1" pad="A"/>
+<wire x1="90.17" y1="26.67" x2="77.618" y2="10.17" width="0" layer="19" extent="1-1"/>
+</signal>
+<signal name="N$7">
+<contactref element="DIODO1" pad="C"/>
+<contactref element="CONTROLBATERIA" pad="B+"/>
+<wire x1="80.01" y1="26.67" x2="38.1" y2="27.305" width="0" layer="19" extent="1-1"/>
+</signal>
 </signals>
